File: photo-relay.brd (EAGLE design)
At the start: 40 x 45 mm, 12 parts, among them IC1 LM393N, K1 351, T1 2N3904, X1 MKDSN1,5/3-5,08, X2 MKDSN1,5/2-5,08

Commit message: fix. transistor connection
Parts:
- R2, R5: value 120K -> 1K
- R6: value 10K -> 1K
Connections:
- removed net N$5: R6.1, T1.2
- net N$1: now also T1.2
- net V+: now also R6.1
Routing:
- net N$1: track 16.1 -> 27.0 mm
- net V+: track 113.2 -> 119.2 mm
- net N$5: track 3.47 -> 0.00 mm
Changed lines of the file:
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@@
 <grid distance="0.5" unitdist="mm" unit="mm" style="lines" multiple="1" display="yes" altdistance="0.025" altunitdist="inch" altunit="inch"/>
 <layers>
-<layer number="1" name="Top" color="4" fill="1" visible="no" active="yes"/>
+<layer number="1" name="Top" color="4" fill="1" visible="yes" active="yes"/>
 <layer number="16" name="Bottom" color="1" fill="1" visible="yes" active="yes"/>
 <layer number="17" name="Pads" color="2" fill="1" visible="yes" active="yes"/>
 <layer number="18" name="Vias" color="2" fill="1" visible="yes" active="yes"/>
-<layer number="19" name="Unrouted" color="6" fill="1" visible="no" active="yes"/>
+<layer number="19" name="Unrouted" color="6" fill="1" visible="yes" active="yes"/>
 <layer number="20" name="Dimension" color="15" fill="1" visible="yes" active="yes"/>
-<layer number="21" name="tPlace" color="7" fill="1" visible="no" active="yes"/>
-<layer number="22" name="bPlace" color="7" fill="1" visible="no" active="yes"/>
-<layer number="23" name="tOrigins" color="15" fill="1" visible="no" active="yes"/>
-<layer number="24" name="bOrigins" color="15" fill="1" visible="no" active="yes"/>
-<layer number="25" name="tNames" color="7" fill="1" visible="no" active="yes"/>
-<layer number="26" name="bNames" color="7" fill="1" visible="no" active="yes"/>
-<layer number="27" name="tValues" color="7" fill="1" visible="no" active="yes"/>
-<layer number="28" name="bValues" color="7" fill="1" visible="no" active="yes"/>
-<layer number="29" name="tStop" color="7" fill="3" visible="no" active="yes"/>
-<layer number="30" name="bStop" color="7" fill="6" visible="no" active="yes"/>
-<layer number="31" name="tCream" color="7" fill="4" visible="no" active="yes"/>
-<layer number="32" name="bCream" color="7" fill="5" visible="no" active="yes"/>
-<layer number="33" name="tFinish" color="6" fill="3" visible="no" active="yes"/>
-<layer number="34" name="bFinish" color="6" fill="6" visible="no" active="yes"/>
-<layer number="35" name="tGlue" color="7" fill="4" visible="no" active="yes"/>
-<layer number="36" name="bGlue" color="7" fill="5" visible="no" active="yes"/>
-<layer number="37" name="tTest" color="7" fill="1" visible="no" active="yes"/>
-<layer number="38" name="bTest" color="7" fill="1" visible="no" active="yes"/>
-<layer number="39" name="tKeepout" color="4" fill="11" visible="no" active="yes"/>
-<layer number="40" name="bKeepout" color="1" fill="11" visible="no" active="yes"/>
-<layer number="41" name="tRestrict" color="4" fill="10" visible="no" active="yes"/>
-<layer number="42" name="bRestrict" color="1" fill="10" visible="no" active="yes"/>
-<layer number="43" name="vRestrict" color="2" fill="10" visible="no" active="yes"/>
-<layer number="44" name="Drills" color="7" fill="1" visible="no" active="yes"/>
-<layer number="45" name="Holes" color="7" fill="1" visible="no" active="yes"/>
-<layer number="46" name="Milling" color="3" fill="1" visible="no" active="yes"/>
-<layer number="47" name="Measures" color="7" fill="1" visible="no" active="yes"/>
-<layer number="48" name="Document" color="7" fill="1" visible="no" active="yes"/>
-<layer number="49" name="Reference" color="7" fill="1" visible="no" active="yes"/>
-<layer number="51" name="tDocu" color="7" fill="1" visible="no" active="yes"/>
-<layer number="52" name="bDocu" color="7" fill="1" visible="no" active="yes"/>
+<layer number="21" name="tPlace" color="7" fill="1" visible="yes" active="yes"/>
+<layer number="22" name="bPlace" color="7" fill="1" visible="yes" active="yes"/>
+<layer number="23" name="tOrigins" color="15" fill="1" visible="yes" active="yes"/>
+<layer number="24" name="bOrigins" color="15" fill="1" visible="yes" active="yes"/>
+<layer number="25" name="tNames" color="7" fill="1" visible="yes" active="yes"/>
+<layer number="26" name="bNames" color="7" fill="1" visible="yes" active="yes"/>
+<layer number="27" name="tValues" color="7" fill="1" visible="yes" active="yes"/>
+<layer number="28" name="bValues" color="7" fill="1" visible="yes" active="yes"/>
+<layer number="29" name="tStop" color="7" fill="3" visible="yes" active="yes"/>
+<layer number="30" name="bStop" color="7" fill="6" visible="yes" active="yes"/>
+<layer number="31" name="tCream" color="7" fill="4" visible="yes" active="yes"/>
+<layer number="32" name="bCream" color="7" fill="5" visible="yes" active="yes"/>
+<layer number="33" name="tFinish" color="6" fill="3" visible="yes" active="yes"/>
+<layer number="34" name="bFinish" color="6" fill="6" visible="yes" active="yes"/>
+<layer number="35" name="tGlue" color="7" fill="4" visible="yes" active="yes"/>
+<layer number="36" name="bGlue" color="7" fill="5" visible="yes" active="yes"/>
+<layer number="37" name="tTest" color="7" fill="1" visible="yes" active="yes"/>
+<layer number="38" name="bTest" color="7" fill="1" visible="yes" active="yes"/>
+<layer number="39" name="tKeepout" color="4" fill="11" visible="yes" active="yes"/>
+<layer number="40" name="bKeepout" color="1" fill="11" visible="yes" active="yes"/>
+<layer number="41" name="tRestrict" color="4" fill="10" visible="yes" active="yes"/>
+<layer number="42" name="bRestrict" color="1" fill="10" visible="yes" active="yes"/>
+<layer number="43" name="vRestrict" color="2" fill="10" visible="yes" active="yes"/>
+<layer number="44" name="Drills" color="7" fill="1" visible="yes" active="yes"/>
+<layer number="45" name="Holes" color="7" fill="1" visible="yes" active="yes"/>
+<layer number="46" name="Milling" color="3" fill="1" visible="yes" active="yes"/>
+<layer number="47" name="Measures" color="7" fill="1" visible="yes" active="yes"/>
+<layer number="48" name="Document" color="7" fill="1" visible="yes" active="yes"/>
+<layer number="49" name="Reference" color="7" fill="1" visible="yes" active="yes"/>
+<layer number="51" name="tDocu" color="7" fill="1" visible="yes" active="yes"/>
+<layer number="52" name="bDocu" color="7" fill="1" visible="yes" active="yes"/>
 <layer number="90" name="Modules" color="5" fill="1" visible="no" active="no"/>
 <layer number="91" name="Nets" color="2" fill="1" visible="no" active="no"/>
@@
 <element name="IC1" library="linear" package="DIL08" value="LM393N" x="33.67" y="21.69"/>
 <element name="R1" library="rcl" package="0204/7" value="Photo" x="15.78" y="11.26"/>
-<element name="R2" library="rcl" package="0204/7" value="120K" x="15.84" y="6.82"/>
+<element name="R2" library="rcl" package="0204/7" value="1K" x="15.84" y="6.82"/>
 <element name="R3" library="rcl" package="0204/7" value="" x="22.87" y="18.19"/>
 <element name="R4" library="rcl" package="RTRIM64W" value="50K" x="24.67" y="8.72"/>
-<element name="R5" library="rcl" package="0204/7" value="120K" x="16.13" y="2.29"/>
-<element name="R6" library="rcl" package="0204/7" value="10K" x="13.5" y="15"/>
+<element name="R5" library="rcl" package="0204/7" value="1K" x="16.13" y="2.29"/>
+<element name="R6" library="rcl" package="0204/7" value="1K" x="13.5" y="15"/>
 <element name="K1" library="relay" package="351" value="351" x="12" y="28">
 <attribute name="OC_NEWARK" value="unknown" x="12" y="28" size="1.778" layer="27" display="off"/>
@@
 <wire x1="4" y1="14.92" x2="3.975" y2="14.92" width="0.4064" layer="16"/>
 <wire x1="3.975" y1="14.92" x2="3.975" y2="7.5189" width="0.4064" layer="16"/>
+<contactref element="R6" pad="1"/>
+<wire x1="9.69" y1="15" x2="9.5" y2="15" width="0.4064" layer="16"/>
+<wire x1="4" y1="14.92" x2="9.69" y2="14.92" width="0.4064" layer="16"/>
+<wire x1="9.69" y1="14.92" x2="9.69" y2="15" width="0.4064" layer="16"/>
 </signal>
 <signal name="V-">
 <contactref element="IC1" pad="4"/>
-</signal>
-<signal name="N$1">
-<contactref element="R3" pad="2"/>
-<contactref element="IC1" pad="1"/>
-<contactref element="R6" pad="2"/>
-<wire x1="17.31" y1="15" x2="26.68" y2="15" width="0.4064" layer="16"/>
-<wire x1="26.68" y1="15" x2="26.68" y2="18.19" width="0.4064" layer="16"/>
-<wire x1="26.68" y1="18.19" x2="29.86" y2="18.19" width="0.4064" layer="16"/>
-<wire x1="29.86" y1="18.19" x2="29.86" y2="17.88" width="0.4064" layer="16"/>
 </signal>
 <signal name="N$2">
@@
 <contactref element="X2" pad="1"/>
 <contactref element="T1" pad="3"/>
-<wire x1="12.32" y1="2.29" x2="12.03" y2="6.82" width="0" layer="19" extent="1-1"/>
+<wire x1="12.03" y1="6.82" x2="12.32" y2="2.29" width="0" layer="19" extent="1-1"/>
 </signal>
 <signal name="N$6">
-</signal>
-<signal name="N$5">
-<contactref element="R6" pad="1"/>
-<wire x1="9.69" y1="15" x2="9.5" y2="15" width="0.4064" layer="16"/>
-<contactref element="T1" pad="2"/>
-<wire x1="9.5" y1="18.095" x2="9.69" y2="18.095" width="0.4064" layer="16"/>
-<wire x1="9.69" y1="18.095" x2="9.69" y2="15" width="0.4064" layer="16"/>
 </signal>
 <signal name="N$8">
@@
 <wire x1="20.9389" y1="31.81" x2="20.9389" y2="40.025" width="1.27" layer="16"/>
 </signal>
+<signal name="N$1">
+<contactref element="T1" pad="2"/>
+<contactref element="R6" pad="2"/>
+<contactref element="R3" pad="2"/>
+<contactref element="IC1" pad="1"/>
+<wire x1="26.68" y1="18.19" x2="29.86" y2="18.19" width="0.4064" layer="16"/>
+<wire x1="29.86" y1="18.19" x2="29.86" y2="17.88" width="0.4064" layer="16"/>
+<wire x1="17.31" y1="15" x2="26.68" y2="15" width="0.4064" layer="16"/>
+<wire x1="26.68" y1="15" x2="26.68" y2="18.19" width="0.4064" layer="16"/>
+<wire x1="17.31" y1="15" x2="13.5" y2="15" width="0.4064" layer="16"/>
+<wire x1="13.5" y1="15" x2="13.5" y2="18" width="0.4064" layer="16"/>
+<wire x1="13.5" y1="18" x2="9.5" y2="18" width="0.4064" layer="16"/>
+<wire x1="9.5" y1="18" x2="9.5" y2="18.095" width="0.4064" layer="16"/>
+</signal>
 </signals>

Commit message: change relay
Parts:
- K1: value 351 -> G5L; device relay:351 -> relay:G5LE
- moved X1 19.5 mm to (4.00, 39.5), turned to 90 degrees
- moved K1 14.0 mm to (23.5, 36.0), turned to 180 degrees
Connections:
- removed net N$10: K1.O1, K1.O2, X1.2
- new net N$5: K1.P, X1.2
- net N$7: now also K1.2; no longer K1.1
- net N$8: now also K1.S, X1.3; no longer K1.P1, K1.P2, X1.1
- net N$9: now also K1.O, X1.1; no longer K1.S1, K1.S2, X1.3
- net V+: now also K1.1; no longer K1.16
Routing:
- net N$5: track 0.00 -> 30.0 mm
- net N$7: track 13.5 -> 41.3 mm
- net N$10: track 15.9 -> 0.00 mm
- net V+: track 119.2 -> 114.3 mm
- net N$8: track 15.9 -> 14.9 mm
- net N$9: track 15.8 -> 16.7 mm
Other:
- board size 40 x 45 mm -> 45 x 45 mm

Commit message: minor fix.
Parts:
- moved K1 0.50 mm to (23.5, 36.5)
Routing:
- net V+: track 114.3 -> 114.8 mm
- net N$9: track 16.7 -> 16.2 mm
- net N$7: track 41.3 -> 41.8 mm
- net N$5: track 30.0 -> 29.5 mm
Changed lines of the file:
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@@
 <grid distance="0.5" unitdist="mm" unit="mm" style="lines" multiple="1" display="yes" altdistance="0.025" altunitdist="inch" altunit="inch"/>
 <layers>
-<layer number="1" name="Top" color="4" fill="1" visible="no" active="yes"/>
+<layer number="1" name="Top" color="4" fill="1" visible="yes" active="yes"/>
 <layer number="16" name="Bottom" color="1" fill="1" visible="yes" active="yes"/>
 <layer number="17" name="Pads" color="2" fill="1" visible="yes" active="yes"/>
 <layer number="18" name="Vias" color="2" fill="1" visible="yes" active="yes"/>
-<layer number="19" name="Unrouted" color="6" fill="1" visible="no" active="yes"/>
+<layer number="19" name="Unrouted" color="6" fill="1" visible="yes" active="yes"/>
 <layer number="20" name="Dimension" color="15" fill="1" visible="yes" active="yes"/>
-<layer number="21" name="tPlace" color="7" fill="1" visible="no" active="yes"/>
-<layer number="22" name="bPlace" color="7" fill="1" visible="no" active="yes"/>
-<layer number="23" name="tOrigins" color="15" fill="1" visible="no" active="yes"/>
-<layer number="24" name="bOrigins" color="15" fill="1" visible="no" active="yes"/>
-<layer number="25" name="tNames" color="7" fill="1" visible="no" active="yes"/>
-<layer number="26" name="bNames" color="7" fill="1" visible="no" active="yes"/>
-<layer number="27" name="tValues" color="7" fill="1" visible="no" active="yes"/>
-<layer number="28" name="bValues" color="7" fill="1" visible="no" active="yes"/>
-<layer number="29" name="tStop" color="7" fill="3" visible="no" active="yes"/>
-<layer number="30" name="bStop" color="7" fill="6" visible="no" active="yes"/>
-<layer number="31" name="tCream" color="7" fill="4" visible="no" active="yes"/>
-<layer number="32" name="bCream" color="7" fill="5" visible="no" active="yes"/>
-<layer number="33" name="tFinish" color="6" fill="3" visible="no" active="yes"/>
-<layer number="34" name="bFinish" color="6" fill="6" visible="no" active="yes"/>
-<layer number="35" name="tGlue" color="7" fill="4" visible="no" active="yes"/>
-<layer number="36" name="bGlue" color="7" fill="5" visible="no" active="yes"/>
-<layer number="37" name="tTest" color="7" fill="1" visible="no" active="yes"/>
-<layer number="38" name="bTest" color="7" fill="1" visible="no" active="yes"/>
-<layer number="39" name="tKeepout" color="4" fill="11" visible="no" active="yes"/>
-<layer number="40" name="bKeepout" color="1" fill="11" visible="no" active="yes"/>
-<layer number="41" name="tRestrict" color="4" fill="10" visible="no" active="yes"/>
-<layer number="42" name="bRestrict" color="1" fill="10" visible="no" active="yes"/>
-<layer number="43" name="vRestrict" color="2" fill="10" visible="no" active="yes"/>
-<layer number="44" name="Drills" color="7" fill="1" visible="no" active="yes"/>
-<layer number="45" name="Holes" color="7" fill="1" visible="no" active="yes"/>
-<layer number="46" name="Milling" color="3" fill="1" visible="no" active="yes"/>
-<layer number="47" name="Measures" color="7" fill="1" visible="no" active="yes"/>
-<layer number="48" name="Document" color="7" fill="1" visible="no" active="yes"/>
-<layer number="49" name="Reference" color="7" fill="1" visible="no" active="yes"/>
-<layer number="51" name="tDocu" color="7" fill="1" visible="no" active="yes"/>
-<layer number="52" name="bDocu" color="7" fill="1" visible="no" active="yes"/>
+<layer number="21" name="tPlace" color="7" fill="1" visible="yes" active="yes"/>
+<layer number="22" name="bPlace" color="7" fill="1" visible="yes" active="yes"/>
+<layer number="23" name="tOrigins" color="15" fill="1" visible="yes" active="yes"/>
+<layer number="24" name="bOrigins" color="15" fill="1" visible="yes" active="yes"/>
+<layer number="25" name="tNames" color="7" fill="1" visible="yes" active="yes"/>
+<layer number="26" name="bNames" color="7" fill="1" visible="yes" active="yes"/>
+<layer number="27" name="tValues" color="7" fill="1" visible="yes" active="yes"/>
+<layer number="28" name="bValues" color="7" fill="1" visible="yes" active="yes"/>
+<layer number="29" name="tStop" color="7" fill="3" visible="yes" active="yes"/>
+<layer number="30" name="bStop" color="7" fill="6" visible="yes" active="yes"/>
+<layer number="31" name="tCream" color="7" fill="4" visible="yes" active="yes"/>
+<layer number="32" name="bCream" color="7" fill="5" visible="yes" active="yes"/>
+<layer number="33" name="tFinish" color="6" fill="3" visible="yes" active="yes"/>
+<layer number="34" name="bFinish" color="6" fill="6" visible="yes" active="yes"/>
+<layer number="35" name="tGlue" color="7" fill="4" visible="yes" active="yes"/>
+<layer number="36" name="bGlue" color="7" fill="5" visible="yes" active="yes"/>
+<layer number="37" name="tTest" color="7" fill="1" visible="yes" active="yes"/>
+<layer number="38" name="bTest" color="7" fill="1" visible="yes" active="yes"/>
+<layer number="39" name="tKeepout" color="4" fill="11" visible="yes" active="yes"/>
+<layer number="40" name="bKeepout" color="1" fill="11" visible="yes" active="yes"/>
+<layer number="41" name="tRestrict" color="4" fill="10" visible="yes" active="yes"/>
+<layer number="42" name="bRestrict" color="1" fill="10" visible="yes" active="yes"/>
+<layer number="43" name="vRestrict" color="2" fill="10" visible="yes" active="yes"/>
+<layer number="44" name="Drills" color="7" fill="1" visible="yes" active="yes"/>
+<layer number="45" name="Holes" color="7" fill="1" visible="yes" active="yes"/>
+<layer number="46" name="Milling" color="3" fill="1" visible="yes" active="yes"/>
+<layer number="47" name="Measures" color="7" fill="1" visible="yes" active="yes"/>
+<layer number="48" name="Document" color="7" fill="1" visible="yes" active="yes"/>
+<layer number="49" name="Reference" color="7" fill="1" visible="yes" active="yes"/>
+<layer number="51" name="tDocu" color="7" fill="1" visible="yes" active="yes"/>
+<layer number="52" name="bDocu" color="7" fill="1" visible="yes" active="yes"/>
 <layer number="90" name="Modules" color="5" fill="1" visible="no" active="no"/>
 <layer number="91" name="Nets" color="2" fill="1" visible="no" active="no"/>
@@
 <element name="D1" library="diode" package="DO35-10" value="1N4148DO35-10" x="4" y="20" rot="R90"/>
 <element name="T1" library="transistor" package="TO92" value="2N3904" x="9.5" y="20" rot="R180"/>
-<element name="K1" library="relay" package="G5LE" value="G5L" x="23.5" y="36" rot="R180">
-<attribute name="MF" value="" x="23.5" y="36" size="1.778" layer="27" rot="R180" display="off"/>
-<attribute name="OC_NEWARK" value="unknown" x="23.5" y="36" size="1.778" layer="27" rot="R180" display="off"/>
-<attribute name="MPN" value="" x="23.5" y="36" size="1.778" layer="27" rot="R180" display="off"/>
-<attribute name="OC_FARNELL" value="unknown" x="23.5" y="36" size="1.778" layer="27" rot="R180" display="off"/>
+<element name="K1" library="relay" package="G5LE" value="G5L" x="23.5" y="36.5" rot="R180">
+<attribute name="MF" value="" x="23.5" y="36.5" size="1.778" layer="27" rot="R180" display="off"/>
+<attribute name="OC_NEWARK" value="unknown" x="23.5" y="36.5" size="1.778" layer="27" rot="R180" display="off"/>
+<attribute name="MPN" value="" x="23.5" y="36.5" size="1.778" layer="27" rot="R180" display="off"/>
+<attribute name="OC_FARNELL" value="unknown" x="23.5" y="36.5" size="1.778" layer="27" rot="R180" display="off"/>
 </element>
 </elements>
@@
 <wire x1="9.69" y1="14.92" x2="9.69" y2="15" width="0.4064" layer="16"/>
 <contactref element="K1" pad="1"/>
-<wire x1="30.993" y1="41.969" x2="37" y2="41.969" width="0.4064" layer="16"/>
-<wire x1="37" y1="41.969" x2="37" y2="27.5" width="0.4064" layer="16"/>
+<wire x1="30.993" y1="42.469" x2="37" y2="42.469" width="0.4064" layer="16"/>
+<wire x1="37" y1="42.469" x2="37" y2="27.5" width="0.4064" layer="16"/>
 <wire x1="37" y1="27.5" x2="29.86" y2="27.5" width="0.4064" layer="16"/>
 <wire x1="29.86" y1="27.5" x2="29.86" y2="25.5" width="0.4064" layer="16"/>
@@
 <contactref element="X2" pad="1"/>
 <contactref element="T1" pad="3"/>
-<wire x1="12.03" y1="6.82" x2="10.77" y2="20" width="0" layer="19" extent="1-1"/>
 </signal>
 <signal name="N$6">
@@
 <wire x1="8.23" y1="20" x2="4" y2="20" width="0.4064" layer="16"/>
 <contactref element="K1" pad="2"/>
-<wire x1="30.993" y1="30.031" x2="24.5" y2="30.031" width="0.4064" layer="16"/>
-<wire x1="24.5" y1="30.031" x2="24.5" y2="25.5" width="0.4064" layer="16"/>
+<wire x1="30.993" y1="30.531" x2="24.5" y2="30.531" width="0.4064" layer="16"/>
+<wire x1="24.5" y1="30.531" x2="24.5" y2="25.5" width="0.4064" layer="16"/>
 <wire x1="24.5" y1="25.5" x2="4" y2="25.5" width="0.4064" layer="16"/>
 <wire x1="4" y1="25.5" x2="4" y2="25.08" width="0.4064" layer="16"/>
@@
 <contactref element="X1" pad="2"/>
 <wire x1="3.975" y1="36.9389" x2="33.025" y2="36.9389" width="0.8128" layer="16"/>
-<wire x1="33.025" y1="36.9389" x2="33.025" y2="36" width="0.8128" layer="16"/>
+<wire x1="33.025" y1="36.9389" x2="33.025" y2="36.5" width="0.8128" layer="16"/>
 </signal>
 <signal name="N$8">
@@
 <contactref element="X1" pad="3"/>
 <wire x1="3.975" y1="42.0189" x2="18.801" y2="42.0189" width="0.8128" layer="16"/>
-<wire x1="18.801" y1="42.0189" x2="18.801" y2="41.969" width="0.8128" layer="16"/>
+<wire x1="18.801" y1="42.0189" x2="18.801" y2="42.469" width="0.8128" layer="16"/>
 </signal>
 <signal name="N$9">
@@
 <contactref element="K1" pad="O"/>
 <wire x1="3.975" y1="31.8589" x2="18.801" y2="31.8589" width="0.8128" layer="16"/>
-<wire x1="18.801" y1="31.8589" x2="18.801" y2="30.031" width="0.8128" layer="16"/>
+<wire x1="18.801" y1="31.8589" x2="18.801" y2="30.531" width="0.8128" layer="16"/>
 </signal>
 </signals>
