File: photo-relay.sch (EAGLE design)
At the start: 11 parts, among them IC1 LM393N, K1 351, Q1 2N3565, X1 MKDSN1,5/3-5,08, X2 MKDSN1,5/2-5,08

Commit message: minor changes
Parts:
- removed Q1: 2N3565, transistor-npn:2N3565
- added D1: 1N4148DO35-10, diode:1N4148DO35-10
- added T1: 2N3904, transistor:2N3904
- R6: value 1K -> 10K
Connections:
- net GND: now also T1.E; no longer Q1.E
- net N$5: now also T1.B; no longer Q1.B
- net N$7: now also D1.A, T1.C; no longer Q1.C
- net V+: now also D1.C
Other:
- moved on the sheet: K1, X1-1, X1-2, X1-3
Changed lines of the file:
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@@
 <layer number="97" name="Info" color="7" fill="1" visible="yes" active="yes"/>
 <layer number="98" name="Guide" color="6" fill="1" visible="yes" active="yes"/>
+<layer number="99" name="SpiceOrder" color="5" fill="1" visible="yes" active="yes"/>
 </layers>
 <schematic xreflabel="%F%N/%S.%C%R" xrefpart="/%S.%C%R">
@@
 <part name="GND2" library="supply1" deviceset="GND" device=""/>
 <part name="GND3" library="supply1" deviceset="GND" device=""/>
-<part name="Q1" library="transistor-npn" deviceset="2N3565" device=""/>
 <part name="GND4" library="supply1" deviceset="GND" device=""/>
-<part name="R6" library="rcl" deviceset="R-EU_" device="0204/7" value="1K"/>
+<part name="R6" library="rcl" deviceset="R-EU_" device="0204/7" value="10K"/>
 <part name="K1" library="relay" deviceset="351" device=""/>
 <part name="X1" library="con-phoenix-508" deviceset="MKDSN1,5/3-5,08" device=""/>
 <part name="X2" library="con-phoenix-508" deviceset="MKDSN1,5/2-5,08" device=""/>
+<part name="D1" library="diode" deviceset="1N4148" device="DO35-10"/>
+<part name="T1" library="transistor" deviceset="2N3904" device=""/>
 </parts>
 <sheets>
@@
 <instance part="GND2" gate="1" x="20.32" y="33.02"/>
 <instance part="GND3" gate="1" x="27.94" y="15.24"/>
-<instance part="Q1" gate="G$1" x="86.36" y="35.56"/>
-<instance part="GND4" gate="1" x="88.9" y="15.24"/>
+<instance part="GND4" gate="1" x="91.44" y="15.24"/>
 <instance part="R6" gate="G$1" x="76.2" y="35.56" rot="R180"/>
-<instance part="K1" gate="1" x="88.9" y="48.26" rot="R180"/>
-<instance part="K1" gate="2" x="104.14" y="48.26"/>
-<instance part="K1" gate="3" x="104.14" y="35.56"/>
-<instance part="X1" gate="-1" x="111.76" y="27.94"/>
-<instance part="X1" gate="-2" x="111.76" y="22.86"/>
-<instance part="X1" gate="-3" x="111.76" y="17.78"/>
+<instance part="K1" gate="1" x="91.44" y="48.26" rot="R180"/>
+<instance part="K1" gate="2" x="106.68" y="48.26"/>
+<instance part="K1" gate="3" x="106.68" y="35.56"/>
+<instance part="X1" gate="-1" x="114.3" y="27.94"/>
+<instance part="X1" gate="-2" x="114.3" y="22.86"/>
+<instance part="X1" gate="-3" x="114.3" y="17.78"/>
 <instance part="X2" gate="-1" x="12.7" y="40.64" rot="R180"/>
 <instance part="X2" gate="-2" x="12.7" y="45.72" rot="R180"/>
+<instance part="D1" gate="G$1" x="76.2" y="45.72" rot="R90"/>
+<instance part="T1" gate="G1" x="88.9" y="35.56"/>
 </instances>
 <busses>
@@
 </segment>
 <segment>
-<pinref part="Q1" gate="G$1" pin="E"/>
 <pinref part="GND4" gate="1" pin="GND"/>
-<wire x1="88.9" y1="30.48" x2="88.9" y2="17.78" width="0.1524" layer="91"/>
+<wire x1="91.44" y1="30.48" x2="91.44" y2="17.78" width="0.1524" layer="91"/>
+<pinref part="T1" gate="G1" pin="E"/>
 </segment>
 </net>
@@
 <pinref part="X2" gate="-2" pin="KL"/>
 <pinref part="K1" gate="1" pin="2"/>
-<wire x1="88.9" y1="53.34" x2="43.18" y2="53.34" width="0.1524" layer="91"/>
+<wire x1="91.44" y1="53.34" x2="76.2" y2="53.34" width="0.1524" layer="91"/>
+<pinref part="D1" gate="G$1" pin="C"/>
+<wire x1="76.2" y1="53.34" x2="43.18" y2="53.34" width="0.1524" layer="91"/>
+<wire x1="76.2" y1="48.26" x2="76.2" y2="53.34" width="0.1524" layer="91"/>
+<junction x="76.2" y="53.34"/>
 </segment>
 </net>
@@
 <segment>
 <pinref part="R6" gate="G$1" pin="1"/>
-<pinref part="Q1" gate="G$1" pin="B"/>
-<wire x1="81.28" y1="35.56" x2="83.82" y2="35.56" width="0.1524" layer="91"/>
+<wire x1="81.28" y1="35.56" x2="86.36" y2="35.56" width="0.1524" layer="91"/>
+<pinref part="T1" gate="G1" pin="B"/>
 </segment>
 </net>
@@
 <segment>
 <pinref part="X1" gate="-1" pin="KL"/>
-<wire x1="109.22" y1="27.94" x2="104.14" y2="27.94" width="0.1524" layer="91"/>
+<wire x1="111.76" y1="27.94" x2="106.68" y2="27.94" width="0.1524" layer="91"/>
 <pinref part="K1" gate="3" pin="P"/>
-<wire x1="104.14" y1="27.94" x2="104.14" y2="33.02" width="0.1524" layer="91"/>
+<wire x1="106.68" y1="27.94" x2="106.68" y2="33.02" width="0.1524" layer="91"/>
 <pinref part="K1" gate="2" pin="P"/>
-<wire x1="104.14" y1="45.72" x2="114.3" y2="45.72" width="0.1524" layer="91"/>
-<wire x1="114.3" y1="45.72" x2="114.3" y2="33.02" width="0.1524" layer="91"/>
-<wire x1="114.3" y1="33.02" x2="104.14" y2="33.02" width="0.1524" layer="91"/>
-<junction x="104.14" y="33.02"/>
+<wire x1="106.68" y1="45.72" x2="116.84" y2="45.72" width="0.1524" layer="91"/>
+<wire x1="116.84" y1="45.72" x2="116.84" y2="33.02" width="0.1524" layer="91"/>
+<wire x1="116.84" y1="33.02" x2="106.68" y2="33.02" width="0.1524" layer="91"/>
+<junction x="106.68" y="33.02"/>
 </segment>
 </net>
@@
 <pinref part="K1" gate="2" pin="S"/>
 <pinref part="K1" gate="3" pin="S"/>
-<wire x1="99.06" y1="53.34" x2="99.06" y2="40.64" width="0.1524" layer="91"/>
-<wire x1="99.06" y1="40.64" x2="99.06" y2="17.78" width="0.1524" layer="91"/>
-<junction x="99.06" y="40.64"/>
+<wire x1="101.6" y1="53.34" x2="101.6" y2="40.64" width="0.1524" layer="91"/>
+<wire x1="101.6" y1="40.64" x2="101.6" y2="17.78" width="0.1524" layer="91"/>
+<junction x="101.6" y="40.64"/>
 <pinref part="X1" gate="-3" pin="KL"/>
-<wire x1="99.06" y1="17.78" x2="109.22" y2="17.78" width="0.1524" layer="91"/>
+<wire x1="101.6" y1="17.78" x2="111.76" y2="17.78" width="0.1524" layer="91"/>
 </segment>
 </net>
 <net name="N$7" class="0">
 <segment>
-<pinref part="Q1" gate="G$1" pin="C"/>
 <pinref part="K1" gate="1" pin="1"/>
-<wire x1="88.9" y1="40.64" x2="88.9" y2="43.18" width="0.1524" layer="91"/>
+<wire x1="91.44" y1="40.64" x2="91.44" y2="43.18" width="0.1524" layer="91"/>
+<pinref part="D1" gate="G$1" pin="A"/>
+<wire x1="76.2" y1="43.18" x2="91.44" y2="43.18" width="0.1524" layer="91"/>
+<junction x="91.44" y="43.18"/>
+<pinref part="T1" gate="G1" pin="C"/>
 </segment>
 </net>
@@
 <pinref part="X1" gate="-2" pin="KL"/>
 <pinref part="K1" gate="3" pin="O"/>
-<wire x1="109.22" y1="22.86" x2="109.22" y2="40.64" width="0.1524" layer="91"/>
+<wire x1="111.76" y1="22.86" x2="111.76" y2="40.64" width="0.1524" layer="91"/>
 <pinref part="K1" gate="2" pin="O"/>
-<wire x1="109.22" y1="40.64" x2="109.22" y2="53.34" width="0.1524" layer="91"/>
-<junction x="109.22" y="40.64"/>
+<wire x1="111.76" y1="40.64" x2="111.76" y2="53.34" width="0.1524" layer="91"/>
+<junction x="111.76" y="40.64"/>
 </segment>
 </net>

Commit message: fix. transistor connection
Parts:
- R2, R5: value 120K -> 1K
- R6: value 10K -> 1K
Connections:
- removed net N$5: R6.1, T1.B
- net N$1: now also T1.B
- net V+: now also R6.1
Other:
- moved on the sheet: D1, K1, R6, T1
Changed lines of the file:
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@@
 <part name="IC1" library="linear" deviceset="LM393" device="N"/>
 <part name="R1" library="rcl" deviceset="R-EU_" device="0204/7" value="Photo"/>
-<part name="R2" library="rcl" deviceset="R-EU_" device="0204/7" value="120K"/>
+<part name="R2" library="rcl" deviceset="R-EU_" device="0204/7" value="1K"/>
 <part name="R3" library="rcl" deviceset="R-EU_" device="0204/7"/>
 <part name="R4" library="rcl" deviceset="R-TRIMM" device="64W" value="50K"/>
-<part name="R5" library="rcl" deviceset="R-EU_" device="0204/7" value="120K"/>
+<part name="R5" library="rcl" deviceset="R-EU_" device="0204/7" value="1K"/>
 <part name="GND1" library="supply1" deviceset="GND" device=""/>
 <part name="GND2" library="supply1" deviceset="GND" device=""/>
 <part name="GND3" library="supply1" deviceset="GND" device=""/>
 <part name="GND4" library="supply1" deviceset="GND" device=""/>
-<part name="R6" library="rcl" deviceset="R-EU_" device="0204/7" value="10K"/>
+<part name="R6" library="rcl" deviceset="R-EU_" device="0204/7" value="1K"/>
 <part name="K1" library="relay" deviceset="351" device=""/>
 <part name="X1" library="con-phoenix-508" deviceset="MKDSN1,5/3-5,08" device=""/>
@@
 <instance part="GND2" gate="1" x="20.32" y="33.02"/>
 <instance part="GND3" gate="1" x="27.94" y="15.24"/>
-<instance part="GND4" gate="1" x="91.44" y="15.24"/>
-<instance part="R6" gate="G$1" x="76.2" y="35.56" rot="R180"/>
-<instance part="K1" gate="1" x="91.44" y="48.26" rot="R180"/>
+<instance part="GND4" gate="1" x="93.98" y="15.24"/>
+<instance part="R6" gate="G$1" x="73.66" y="40.64" rot="R270"/>
+<instance part="K1" gate="1" x="93.98" y="48.26" rot="R180"/>
 <instance part="K1" gate="2" x="106.68" y="48.26"/>
 <instance part="K1" gate="3" x="106.68" y="35.56"/>
@@
 <instance part="X2" gate="-1" x="12.7" y="40.64" rot="R180"/>
 <instance part="X2" gate="-2" x="12.7" y="45.72" rot="R180"/>
-<instance part="D1" gate="G$1" x="76.2" y="45.72" rot="R90"/>
-<instance part="T1" gate="G1" x="88.9" y="35.56"/>
+<instance part="D1" gate="G$1" x="78.74" y="45.72" rot="R90"/>
+<instance part="T1" gate="G1" x="91.44" y="35.56"/>
 </instances>
 <busses>
 </busses>
 <nets>
-<net name="N$1" class="0">
-<segment>
-<pinref part="R3" gate="G$1" pin="2"/>
-<pinref part="IC1" gate="A" pin="OUT"/>
-<wire x1="63.5" y1="48.26" x2="68.58" y2="48.26" width="0.1524" layer="91"/>
-<wire x1="68.58" y1="48.26" x2="68.58" y2="35.56" width="0.1524" layer="91"/>
-<pinref part="R6" gate="G$1" pin="2"/>
-<wire x1="68.58" y1="35.56" x2="71.12" y2="35.56" width="0.1524" layer="91"/>
-<junction x="68.58" y="35.56"/>
-</segment>
-</net>
 <net name="N$2" class="0">
 <segment>
@@
 <segment>
 <pinref part="GND4" gate="1" pin="GND"/>
-<wire x1="91.44" y1="30.48" x2="91.44" y2="17.78" width="0.1524" layer="91"/>
+<wire x1="93.98" y1="30.48" x2="93.98" y2="17.78" width="0.1524" layer="91"/>
 <pinref part="T1" gate="G1" pin="E"/>
 </segment>
@@
 <pinref part="X2" gate="-2" pin="KL"/>
 <pinref part="K1" gate="1" pin="2"/>
-<wire x1="91.44" y1="53.34" x2="76.2" y2="53.34" width="0.1524" layer="91"/>
+<wire x1="93.98" y1="53.34" x2="78.74" y2="53.34" width="0.1524" layer="91"/>
 <pinref part="D1" gate="G$1" pin="C"/>
-<wire x1="76.2" y1="53.34" x2="43.18" y2="53.34" width="0.1524" layer="91"/>
-<wire x1="76.2" y1="48.26" x2="76.2" y2="53.34" width="0.1524" layer="91"/>
-<junction x="76.2" y="53.34"/>
-</segment>
-</net>
-<net name="N$5" class="0">
-<segment>
+<wire x1="78.74" y1="53.34" x2="73.66" y2="53.34" width="0.1524" layer="91"/>
+<wire x1="73.66" y1="53.34" x2="43.18" y2="53.34" width="0.1524" layer="91"/>
+<wire x1="78.74" y1="48.26" x2="78.74" y2="53.34" width="0.1524" layer="91"/>
+<junction x="78.74" y="53.34"/>
 <pinref part="R6" gate="G$1" pin="1"/>
-<wire x1="81.28" y1="35.56" x2="86.36" y2="35.56" width="0.1524" layer="91"/>
-<pinref part="T1" gate="G1" pin="B"/>
+<wire x1="73.66" y1="45.72" x2="73.66" y2="53.34" width="0.1524" layer="91"/>
+<junction x="73.66" y="53.34"/>
 </segment>
 </net>
@@
 <segment>
 <pinref part="K1" gate="1" pin="1"/>
-<wire x1="91.44" y1="40.64" x2="91.44" y2="43.18" width="0.1524" layer="91"/>
+<wire x1="93.98" y1="40.64" x2="93.98" y2="43.18" width="0.1524" layer="91"/>
 <pinref part="D1" gate="G$1" pin="A"/>
-<wire x1="76.2" y1="43.18" x2="91.44" y2="43.18" width="0.1524" layer="91"/>
-<junction x="91.44" y="43.18"/>
+<wire x1="78.74" y1="43.18" x2="93.98" y2="43.18" width="0.1524" layer="91"/>
+<junction x="93.98" y="43.18"/>
 <pinref part="T1" gate="G1" pin="C"/>
 </segment>
@@
 </segment>
 </net>
+<net name="N$1" class="0">
+<segment>
+<pinref part="T1" gate="G1" pin="B"/>
+<pinref part="R6" gate="G$1" pin="2"/>
+<wire x1="73.66" y1="35.56" x2="88.9" y2="35.56" width="0.1524" layer="91"/>
+<junction x="73.66" y="35.56"/>
+<pinref part="IC1" gate="A" pin="OUT"/>
+<pinref part="R3" gate="G$1" pin="2"/>
+<wire x1="63.5" y1="48.26" x2="68.58" y2="48.26" width="0.1524" layer="91"/>
+<wire x1="68.58" y1="48.26" x2="68.58" y2="35.56" width="0.1524" layer="91"/>
+<wire x1="68.58" y1="35.56" x2="73.66" y2="35.56" width="0.1524" layer="91"/>
+<junction x="68.58" y="35.56"/>
+</segment>
+</net>

Commit message: change relay
Parts:
- K1: value 351 -> G5L; device relay:351 -> relay:G5L
Connections:
- removed net N$10: K12.O, K13.O, X1-2.KL
- new net N$5: K12.P, X1-2.KL
- net N$7: now also K11.2; no longer K11.1
- net N$8: now also K12.S, X1-3.KL; no longer K12.P, K13.P, X1-1.KL
- net N$9: now also K12.O, X1-1.KL; no longer K12.S, K13.S, X1-3.KL
- net V+: now also K11.1; no longer K11.2
Other:
- moved on the sheet: K1
Changed lines of the file:
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@@
 <part name="GND4" library="supply1" deviceset="GND" device=""/>
 <part name="R6" library="rcl" deviceset="R-EU_" device="0204/7" value="1K"/>
-<part name="K1" library="relay" deviceset="351" device=""/>
 <part name="X1" library="con-phoenix-508" deviceset="MKDSN1,5/3-5,08" device=""/>
 <part name="X2" library="con-phoenix-508" deviceset="MKDSN1,5/2-5,08" device=""/>
 <part name="D1" library="diode" deviceset="1N4148" device="DO35-10"/>
 <part name="T1" library="transistor" deviceset="2N3904" device=""/>
+<part name="K1" library="relay" deviceset="G5L" device=""/>
 </parts>
 <sheets>
@@
 <instance part="GND4" gate="1" x="93.98" y="15.24"/>
 <instance part="R6" gate="G$1" x="73.66" y="40.64" rot="R270"/>
-<instance part="K1" gate="1" x="93.98" y="48.26" rot="R180"/>
-<instance part="K1" gate="2" x="106.68" y="48.26"/>
-<instance part="K1" gate="3" x="106.68" y="35.56"/>
 <instance part="X1" gate="-1" x="114.3" y="27.94"/>
 <instance part="X1" gate="-2" x="114.3" y="22.86"/>
@@
 <instance part="D1" gate="G$1" x="78.74" y="45.72" rot="R90"/>
 <instance part="T1" gate="G1" x="91.44" y="35.56"/>
+<instance part="K1" gate="1" x="93.98" y="48.26"/>
+<instance part="K1" gate="2" x="106.68" y="48.26"/>
 </instances>
 <busses>
@@
 <junction x="43.18" y="45.72"/>
 <pinref part="X2" gate="-2" pin="KL"/>
-<pinref part="K1" gate="1" pin="2"/>
 <wire x1="93.98" y1="53.34" x2="78.74" y2="53.34" width="0.1524" layer="91"/>
 <pinref part="D1" gate="G$1" pin="C"/>
@@
 <wire x1="73.66" y1="45.72" x2="73.66" y2="53.34" width="0.1524" layer="91"/>
 <junction x="73.66" y="53.34"/>
-</segment>
-</net>
-<net name="N$8" class="0">
-<segment>
-<pinref part="X1" gate="-1" pin="KL"/>
-<wire x1="111.76" y1="27.94" x2="106.68" y2="27.94" width="0.1524" layer="91"/>
-<pinref part="K1" gate="3" pin="P"/>
-<wire x1="106.68" y1="27.94" x2="106.68" y2="33.02" width="0.1524" layer="91"/>
-<pinref part="K1" gate="2" pin="P"/>
-<wire x1="106.68" y1="45.72" x2="116.84" y2="45.72" width="0.1524" layer="91"/>
-<wire x1="116.84" y1="45.72" x2="116.84" y2="33.02" width="0.1524" layer="91"/>
-<wire x1="116.84" y1="33.02" x2="106.68" y2="33.02" width="0.1524" layer="91"/>
-<junction x="106.68" y="33.02"/>
-</segment>
-</net>
-<net name="N$9" class="0">
-<segment>
-<pinref part="K1" gate="2" pin="S"/>
-<pinref part="K1" gate="3" pin="S"/>
-<wire x1="101.6" y1="53.34" x2="101.6" y2="40.64" width="0.1524" layer="91"/>
-<wire x1="101.6" y1="40.64" x2="101.6" y2="17.78" width="0.1524" layer="91"/>
-<junction x="101.6" y="40.64"/>
-<pinref part="X1" gate="-3" pin="KL"/>
-<wire x1="101.6" y1="17.78" x2="111.76" y2="17.78" width="0.1524" layer="91"/>
+<pinref part="K1" gate="1" pin="1"/>
 </segment>
 </net>
 <net name="N$7" class="0">
 <segment>
-<pinref part="K1" gate="1" pin="1"/>
 <wire x1="93.98" y1="40.64" x2="93.98" y2="43.18" width="0.1524" layer="91"/>
 <pinref part="D1" gate="G$1" pin="A"/>
 <wire x1="78.74" y1="43.18" x2="93.98" y2="43.18" width="0.1524" layer="91"/>
+<pinref part="T1" gate="G1" pin="C"/>
+<pinref part="K1" gate="1" pin="2"/>
 <junction x="93.98" y="43.18"/>
-<pinref part="T1" gate="G1" pin="C"/>
-</segment>
-</net>
-<net name="N$10" class="0">
-<segment>
-<pinref part="X1" gate="-2" pin="KL"/>
-<pinref part="K1" gate="3" pin="O"/>
-<wire x1="111.76" y1="22.86" x2="111.76" y2="40.64" width="0.1524" layer="91"/>
-<pinref part="K1" gate="2" pin="O"/>
-<wire x1="111.76" y1="40.64" x2="111.76" y2="53.34" width="0.1524" layer="91"/>
-<junction x="111.76" y="40.64"/>
 </segment>
 </net>
@@
 </segment>
 </net>
+<net name="N$5" class="0">
+<segment>
+<pinref part="K1" gate="2" pin="P"/>
+<wire x1="106.68" y1="45.72" x2="106.68" y2="22.86" width="0.1524" layer="91"/>
+<pinref part="X1" gate="-2" pin="KL"/>
+<wire x1="106.68" y1="22.86" x2="111.76" y2="22.86" width="0.1524" layer="91"/>
+</segment>
+</net>
+<net name="N$8" class="0">
+<segment>
+<pinref part="K1" gate="2" pin="S"/>
+<wire x1="101.6" y1="53.34" x2="101.6" y2="17.78" width="0.1524" layer="91"/>
+<pinref part="X1" gate="-3" pin="KL"/>
+<wire x1="101.6" y1="17.78" x2="111.76" y2="17.78" width="0.1524" layer="91"/>
+</segment>
+</net>
+<net name="N$9" class="0">
+<segment>
+<pinref part="X1" gate="-1" pin="KL"/>
+<pinref part="K1" gate="2" pin="O"/>
+<wire x1="111.76" y1="27.94" x2="111.76" y2="53.34" width="0.1524" layer="91"/>
+</segment>
+</net>
